File: Hardware/rev100/I2C_SPI_to_USB.kicad_sch (KiCad schematic)
At the start: 50 parts

Commit message: Included USB ports on schematic
Connections:
- no-connect marks 19 -> 23
Changed lines of the file:
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@@
   (title_block
     (title "Electronics Multitool - I2C_SPI_to_USB")
+    (rev "100")
   )
   (junction (at 71.12 175.26) (diameter 0) (color 0 0 0 0)
@@
   (no_connect (at 128.27 149.86))
   (no_connect (at 128.27 152.4))
+  (no_connect (at 39.37 151.13))
+  (no_connect (at 39.37 146.05))
+  (no_connect (at 40.64 63.5))
+  (no_connect (at 40.64 58.42))
   (wire (pts (xy 85.09 144.78) (xy 85.09 146.05))
     (stroke (width 0) (type default) (color 0 0 0 0))
