File: Hardware/rev100/Serial_to_USB.kicad_sch (KiCad schematic)
At the start: 16 parts

Commit message: Included USB ports on schematic
Connections:
- net 3V3 renamed 3V3_Serial
- no-connect marks 11 -> 13
Changed lines of the file:
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@@
   (title_block
     (title "Electronics Multitool - Serial to USB")
+    (rev "100")
   )
   (junction (at 116.84 110.49) (diameter 0) (color 0 0 0 0)
@@
   )
   (no_connect (at 213.36 86.36))
+  (no_connect (at 72.39 102.87))
+  (no_connect (at 72.39 107.95))
   (no_connect (at 149.86 105.41))
   (no_connect (at 149.86 107.95))
@@
     (stroke (width 0) (type default) (color 0 0 0 0))
   )
-  (wire (pts (xy 110.49 102.87) (xy 118.11 102.87))
+  (wire (pts (xy 107.95 102.87) (xy 118.11 102.87))
     (stroke (width 0) (type default) (color 0 0 0 0))
   )
@@
     (effects (font (size 1.27 1.27)) (justify left bottom))
   )
-  (label "3V3" (at 105.41 83.82 0)
+  (label "3V3_Serial" (at 102.87 83.82 0)
     (effects (font (size 1.27 1.27)) (justify left bottom))
   )
@@
     (effects (font (size 1.27 1.27)) (justify left bottom))
   )
-  (label "3V3" (at 111.76 102.87 0)
-    (effects (font (size 1.27 1.27)) (justify left bottom))
-  )
+  (label "3V3_Serial" (at 107.95 102.87 0)
+    (effects (font (size 1.27 1.27)) (justify left bottom))
+  )
